File: RP2040-Bridge-CAN-SPI.kicad_sch (KiCad schematic)
At the start: 0 parts

Commit message: update design
Other:
- sheet SPI-Interface renamed Mikro-Interface
Changed lines of the file:
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@@
 			(color 0 0 0 0.0000)
 		)
-		(property "Sheetname" "SPI-Interface"
+		(property "Sheetname" "Mikro-Interface"
 			(at 170.18 64.0584 0)
 			(effects
