File: spi.kicad_sch (KiCad schematic)
At the start: 0 parts

Commit message: update design
Parts:
- added J2, J3: Conn_01x08_Socket, Connector_PinSocket_2.54mm:PinSocket_1x08_P2.54mm_Vertical, symbol Connector:Conn_01x08_Socket
- added R4, R5: 10K, Resistor_SMD:R_0603_1608Metric_Pad0.98x0.95mm_HandSolder, symbol Device:R_Small
- added R6, R7: 4K7, Resistor_SMD:R_0603_1608Metric_Pad0.98x0.95mm_HandSolder, symbol Device:R_Small
- added U4: AT24CS01-SSHM, Package_SO:SOIC-8_3.9x4.9mm_P1.27mm, symbol Memory_EEPROM:AT24CS01-SSHM
Connections:
- new net: R4.2, U4.1 (A0)
- new net: R5.1, U4.7 (WP)
- new net +3V3: J2.7 (Pin_7), R4.1, R6.2, R7.2, U4.8 (VCC)
- new net ADCIN0: J2.1 (Pin_1)
- new net GND: J2.8 (Pin_8), J3.8 (Pin_8), R5.2, U4.2 (A1), U4.3 (A2), U4.4 (GND)
- new net I2C0_SCL: J3.5 (Pin_5)
- new net I2C0_SDA: J3.6 (Pin_6)
- new net I2C1_SCL: R7.1, U4.6 (SCL)
- new net I2C1_SDA: R6.1, U4.5 (SDA)
- new net MIKRO_INT: J3.2 (Pin_2)
- new net MIKRO_PWM: J3.1 (Pin_1)
- new net MIKRO_RST: J2.2 (Pin_2)
- new net SPI1_CS: J2.3 (Pin_3)
- new net SPI1_RX: J2.5 (Pin_5)
- new net SPI1_SCK: J2.4 (Pin_4)
- new net SPI1_TX: J2.6 (Pin_6)
- new net UART1_RX: J3.4 (Pin_4)
- new net UART1_TX: J3.3 (Pin_3)
- new net VCC: J3.7 (Pin_7)
