File: RP2040-Bridge-CAN-SPI.kicad_pcb (KiCad board)
At the start: 2 copper layers, 87.6 x 54.6 mm, 30 parts, among them J1 Conn_01x03_Socket, J2 Conn_01x08_Socket, J3 Conn_01x08_Socket, U1 Pico, U2 High-speed CAN FD Transceiver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, U3 MCP2517FD-xSL, U4 AT24CS01-SSHM, Y1 40MHz

Commit message: updates
Other:
- board text added: "0"
- board text added: "0 mm"
- board text added: "0.00 mils / 0.00 mils"
- board text added: "0.01 mm"
- board text added: "0.02"
- board text added: "0.035 mm"
- board text added: "1"
- board text added: "1.51 mm"
- board text added: "11.81 mils"
- board text added: "2"
- board text added: "3.3"
- board text added: "3450.00 mils x 2150.00 mils"
- board text added: "4.5"
- board text added: "62.99 mils"
- board text added: "B.Cu"
- board text added: "B.Mask"
- board text added: "B.Paste"
- board text added: "B.Silkscreen"
- board text added: "BOARD CHARACTERISTICS"
- board text added: "Bottom Silk Screen"
- board text added: "Bottom Solder Mask"
- board text added: "Bottom Solder Paste"
- board text added: "Epsilon R"
- board text added: "F.Cu"
- board text added: "F.Mask"
- board text added: "F.Paste"
- board text added: "F.Silkscreen"
- board text added: "FR4"
- board text added: "Loss Tangent"
- board text added: "None"
- board text added: "Not specified"
- board text added: "Top Silk Screen"
- board text added: "Top Solder Mask"
- board text added: "Top Solder Paste"
- board text added: "copper"
- board text added: "core"
- board text added: "介质"
- board text added: "厚度 (mm)"
- board text added: "否"
- board text added: "存在半孔焊盘:"
- board text added: "层名称"
- board text added: "最小孔径:"
- board text added: "最小走线/间距:"
- board text added: "材料"
- board text added: "板厚:"
- board text added: "板子整体尺寸:"
- board text added: "板边倒角处理:"
- board text added: "类型"
- board text added: "铜层数量:"
- board text added: "镀铜处理:"
- board text added: "阻抗控制:"
- board text added: "需要电镀板边:"
- board text added: "颜色"
