File: can_fd.kicad_sch (KiCad schematic)
At the start: 0 parts

Commit message: update design
Parts:
- added C1: 22uF, Capacitor_SMD:C_0805_2012Metric_Pad1.18x1.45mm_HandSolder, symbol Device:C_Small
- added C10, C2: 1uF, Capacitor_SMD:C_0603_1608Metric_Pad1.08x0.95mm_HandSolder, symbol Device:C_Small
- added C11, C5, C6: 100nF, Capacitor_SMD:C_0603_1608Metric_Pad1.08x0.95mm_HandSolder, symbol Device:C_Small
- added C3, C4: 47pF, Capacitor_SMD:C_0603_1608Metric_Pad1.08x0.95mm_HandSolder, symbol Device:C_Small
- added C7: 4700pF, Capacitor_SMD:C_0603_1608Metric_Pad1.08x0.95mm_HandSolder, symbol Device:C_Small
- added C8, C9: 22pF, Capacitor_SMD:C_0603_1608Metric_Pad1.08x0.95mm_HandSolder, symbol Device:C_Small
- added D1: ESDCAN24-2BLY, Package_TO_SOT_SMD:SOT-23-3, symbol Device:D_TVS_Dual_AAC
- added J1: Conn_01x03_Socket, TerminalBlock:TerminalBlock_bornier-3_P5.08mm, symbol Connector:Conn_01x03_Socket
- added JP1, JP2: Jumper_2_Small_Open, Connector_PinHeader_2.00mm:PinHeader_1x02_P2.00mm_Vertical, symbol Jumper:Jumper_2_Small_Open
- added R1: 10K, Resistor_SMD:R_0603_1608Metric_Pad0.98x0.95mm_HandSolder, symbol Device:R_Small
- added R2, R3: 60.4, Resistor_SMD:R_0603_1608Metric_Pad0.98x0.95mm_HandSolder, symbol Device:R_Small
- added TP1: TestPoint, TestPoint:TestPoint_Pad_D1.0mm, symbol Connector:TestPoint
- added U2: High-speed CAN FD Transceiver with Standby Mode a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, Package_SO:SOIC-8_3.9x4.9mm_P1.27mm, symbol Interface_CAN_LIN:ATA6563-GAQWx
- added U3: MCP2517FD-xSL, Package_SO:SOIC-14_3.9x8.7mm_P1.27mm, symbol Interface_CAN_LIN:MCP2518FD-xSL
- added Y1: 40MHz, Crystal:Crystal_SMD_SeikoEpson_TSX3225-4Pin_3.2x2.5mm, symbol Device:Crystal_GND24_Small
Connections:
- new net: TP1.1, U3.3 (CLKO/SOF)
- new net: C8.1, U3.5 (OSC2), Y1.1
- new net: C9.1, U3.6 (OSC1), Y1.3
- new net: C7.1, R2.1, R3.1
- new net: JP1.2 (B), R3.2
- new net: JP2.2 (B), R2.2
- new net +3V3: C10.1, C11.1, C2.1, C6.1, U2.5 (VIO), U3.14 (VDD)
- new net CANH: C3.1, D1.2 (A2), J1.3 (Pin_3), JP1.1 (A), U2.7 (CANH)
- new net CANL: C4.1, D1.1 (A1), J1.2 (Pin_2), JP2.1 (A), U2.6 (CANL)
- new net CAN_INT: U3.4 (~{INT})
- new net CAN_RX_INT: U3.8 (~{INT1}/GPIO1)
- new net CAN_TX_INT: U3.9 (~{INT0}/GPIO0/XSTBY)
- new net GND: C1.2, C10.2, C11.2, C2.2, C3.2, C4.2, C5.2, C6.2, C7.2, C8.2, C9.2, D1.3 (common), J1.1 (Pin_1), R1.2, U2.2 (GND), U3.7 (VSS), Y1.2, Y1.4
- new net GPIO26: R1.1, U2.8 (STBY)
- new net RXCAN: U2.4 (RXD), U3.2 (RXCAN)
- new net SPI0_CS: U3.13 (~{CS})
- new net SPI0_RX: U3.12 (SDO)
- new net SPI0_SCK: U3.10 (SCK)
- new net SPI0_TX: U3.11 (SDI)
- new net TXCAN: U2.1 (TXD), U3.1 (TXCAN)
- new net VCC: C1.1, C5.1, U2.3 (VCC)

Commit message: updates
Changed lines of the file:
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@@
 (kicad_sch
-	(version 20231120)
+	(version 20250114)
 	(generator "eeschema")
-	(generator_version "8.0")
+	(generator_version "9.0")
 	(paper "A4")
 	(junction
@@
 	(label "RXCAN"
 		(at 172.72 99.06 0)
-		(fields_autoplaced yes)
 		(effects
 			(font
@@
 	(label "CAN_RX_INT"
 		(at 172.72 114.3 0)
-		(fields_autoplaced yes)
 		(effects
 			(font
@@
 	(label "CANL"
 		(at 58.42 45.72 0)
-		(fields_autoplaced yes)
 		(effects
 			(font
@@
 	(label "CANL"
 		(at 86.36 104.14 0)
-		(fields_autoplaced yes)
 		(effects
 			(font
@@
 	(label "CANH"
 		(at 58.42 43.18 0)
-		(fields_autoplaced yes)
 		(effects
 			(font
@@
 	(label "CAN_INT"
 		(at 172.72 109.22 0)
-		(fields_autoplaced yes)
 		(effects
 			(font
@@
 	(label "RXCAN"
 		(at 57.15 106.68 0)
-		(fields_autoplaced yes)
 		(effects
 			(font
@@
 	(label "CAN_TX_INT"
 		(at 172.72 111.76 0)
-		(fields_autoplaced yes)
 		(effects
 			(font
@@
 	(label "CANH"
 		(at 86.36 101.6 0)
-		(fields_autoplaced yes)
 		(effects
 			(font
@@
 	(label "TXCAN"
 		(at 57.15 99.06 0)
-		(fields_autoplaced yes)
 		(effects
 			(font
@@
 	(label "TXCAN"
 		(at 172.72 101.6 0)
-		(fields_autoplaced yes)
-		(effects
-			(font
+		(effects
+			(font
